File: kicad/cpld_atmega/cpld_atmega.sch (KiCad schematic (older format))
At the start: 33 parts, among them CON1 AVR-ISP-6, J1 PWR, J10 FB 4, J2 ADC, J3 Port B, J4 PORT D, J5 Port C, J6 FB 1, J7 FB 2, J8 JTAG, J9 FB 3, SW1 SW_Push, SW2 PWR, U1 LM1117-3.3, U2 ATMEGA168A-AU, U3 XC9572XL-VQFP44, Y1 12Mhz

Commit message: label s are added
Parts:
- added MK1, MK2: MH, MountingHole:MountingHole_2.5mm_Pad, symbol Mechanical:Mounting_Hole_PAD
- R3: value 4k7 -> 10k
Connections:
- net labels added: GNDPWR
- wire segments 178 -> 183

Commit message: version 0.1
Parts:
- removed C5: 100n, Capacitors_THT:C_Disc_D4.3mm_W1.9mm_P5.00mm, symbol device:C_Small
- removed D1: TL431D, Housings_SOIC:SOIC-8_3.9x4.9mm_Pitch1.27mm, symbol references:TL431D
- removed J10: FB 4, Pin_Headers:Pin_Header_Straight_1x08_Pitch2.54mm, symbol Connector:Conn_01x08
- removed J2: ADC, Pin_Headers:Pin_Header_Straight_1x03_Pitch2.54mm, symbol Connector:Conn_01x03
- removed J3: Port B, Pin_Headers:Pin_Header_Straight_1x08_Pitch2.54mm, symbol Connector:Conn_01x08
- removed J4: PORT D, Pin_Headers:Pin_Header_Straight_1x10_Pitch2.54mm, symbol Connector:Conn_01x10
- removed J5: Port C, Pin_Headers:Pin_Header_Straight_1x08_Pitch2.54mm, symbol Connector:Conn_01x08
- removed J6: FB 1, Pin_Headers:Pin_Header_Straight_1x04_Pitch2.54mm, symbol Connector:Conn_01x04
- removed J7: FB 2, Pin_Headers:Pin_Header_Straight_1x10_Pitch2.54mm, symbol Connector:Conn_01x10
- removed J8: JTAG, Pin_Headers:Pin_Header_Straight_2x05_Pitch2.54mm, symbol Connector:Conn_02x05_Odd_Even
- removed J9: FB 3, Pin_Headers:Pin_Header_Straight_1x09_Pitch2.54mm, symbol Connector:Conn_01x09
- removed R3: 10k, Resistors_SMD:R_1206, symbol device:R_Small
- removed U3: XC9572XL-VQFP44, Housings_QFP:LQFP-44_10x10mm_Pitch0.8mm, symbol xc9572xl:XC9572XL-VQFP44
- added C3: 100n, Capacitor_SMD:C_0805_2012Metric_Pad1.15x1.40mm_HandSolder, symbol cpld_atmega-rescue:C_Small-device
- added D1: LED, LED_SMD:LED_1206_3216Metric_Pad1.42x1.75mm_HandSolder, symbol Device:LED
- added J10, J11, J6, J9: Conn_01x11, Connector_PinSocket_2.54mm:PinSocket_1x11_P2.54mm_Vertical, symbol Connector_Generic:Conn_01x11
- added J12: JTAG, Connector_PinSocket_2.54mm:PinSocket_1x07_P2.54mm_Vertical, symbol Connector_Generic:Conn_01x07
- added J2, J3, J4, J5: Conn_01x08_Male, Connector_PinSocket_2.54mm:PinSocket_1x08_P2.54mm_Vertical, symbol Connector:Conn_01x08_Male
- added J7: CLOCK, Connector_PinSocket_2.54mm:PinSocket_1x03_P2.54mm_Vertical, symbol Connector_Generic:Conn_01x03
- added R3: 1k, Resistor_SMD:R_0603_1608Metric_Pad1.05x0.95mm_HandSolder, symbol cpld_atmega-rescue:R_Small-device
- added R8: 470, Resistor_SMD:R_0603_1608Metric_Pad1.05x0.95mm_HandSolder, symbol cpld_atmega-rescue:R_Small-device
- added U3: XC9572XL-VQFP44, Package_QFP:LQFP-44_10x10mm_P0.8mm, symbol cpld_atmega-rescue:XC9572XL-VQFP44-SQ
- C1, C2, C7: symbol device:C_Small -> cpld_atmega-rescue:C_Small-device
- C4, C9: footprint Capacitors_SMD:C_0805_HandSoldering -> Capacitor_SMD:C_0805_2012Metric_Pad1.15x1.40mm_HandSolder; symbol device:C_Small -> cpld_atmega-rescue:C_Small-device
- C6, C8: symbol device:CP_Small -> cpld_atmega-rescue:CP_Small-device
- CON1: symbol atmel:AVR-ISP-6 -> cpld_atmega-rescue:AVR-ISP-6-atmel
- J1: footprint Connectors_Hirose:Hirose_DF63-2P-3.96DSA_02x3.96mm_Straight -> TerminalBlock_RND:TerminalBlock_RND_205-00001_1x02_P5.00mm_Horizontal; symbol Connector:Conn_01x02 -> cpld_atmega-rescue:Conn_01x02-Connector
- MK1, MK2: symbol Mechanical:Mounting_Hole_PAD -> cpld_atmega-rescue:Mounting_Hole_PAD-Mechanical
- R1: value 1k -> 0; footprint Resistors_SMD:R_1206 -> Resistor_SMD:R_0805_2012Metric_Pad1.15x1.40mm_HandSolder; symbol device:R_Small -> cpld_atmega-rescue:R_Small-device
- R2: value 4k7 -> 10K; footprint Resistors_SMD:R_1206 -> Resistor_SMD:R_0603_1608Metric_Pad1.05x0.95mm_HandSolder; symbol device:R_Small -> cpld_atmega-rescue:R_Small-device
- R4, R5, R6: footprint Resistors_SMD:R_1206 -> Resistor_SMD:R_0603_1608Metric_Pad1.05x0.95mm_HandSolder; symbol device:R_Small -> cpld_atmega-rescue:R_Small-device
- R7: value 4k7 -> 1K; footprint Resistors_SMD:R_1206 -> Resistor_SMD:R_0603_1608Metric_Pad1.05x0.95mm_HandSolder; symbol device:R_Small -> cpld_atmega-rescue:R_Small-device
- SW2: symbol sw_dpdt_x2:SW_DPDT_x2 -> cpld_atmega-rescue:SW_DPDT_x2-sw_dpdt_x2
- U1: symbol regul:LM1117-1.8 -> cpld_atmega-rescue:LM1117-1.8-regul
- U2: symbol atmel:ATMEGA168A-AU -> cpld_atmega-rescue:ATMEGA168A-AU-atmel
- Y1: symbol device:Crystal_Small -> cpld_atmega-rescue:Crystal_Small-device
Connections:
- net labels added: P1, P10, P11, P12, P13, P14, P15, P16, P17, P18, P19, P2, P20, P21, P22, P23, P24, P25, P26, P27, P28, P3, P30, P31, P32, P4, P5, P6, P7, P8, P9
- net labels removed: +2V5, GNDPWR, MISO_, MOSI_, PC0, PC1, PC2, PC3, PC4, PC5, SCK_
- wire segments 183 -> 198
- no-connect marks 5 -> 3
Other:
- moved on the sheet: SW1
